File: Power_Supply/Power_Supply.kicad_pcb (KiCad board)
At the start: 2 copper layers, 50 x 100 mm, 34 parts, among them J1 Cable_PAD, J2 Cable_PAD, J4 CONN_01X03, J5 jack, Q1 TIP41C, Q2 BD139, Q3 BC548, Q4 BC558, Q5 BC558, SW1 SW_SPST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

Commit message: new
Parts:
- added J3: Cable_PAD, EESTN5:Separador_M3_10mm, F.Cu at (155.0, 45.0)
- added J6: Cable_PAD, EESTN5:Separador_M3_10mm, F.Cu at (195.0, 45.0)
- added J7: Cable_PAD, EESTN5:Separador_M3_10mm, F.Cu at (155.0, 135.0)
- added J8: Cable_PAD, EESTN5:Separador_M3_10mm, F.Cu at (195.0, 135.0)
- added JP3: Jumper, Modified_Footprints:JUMPER, B.Cu at (162.1, 122.0)
- R2, R6: footprint EESTN5:Potenciometro -> EESTN5:Pin_Header_3
- SW1: footprint EESTN5:BORNERA2 -> EESTN5:Pin_Header_2
- moved J4 111.2 mm to (156.5, 126.0)
- moved SW2 110.5 mm to (169.5, 134.5)
- moved R1 109.8 mm to (181.5, 74.5)
- moved U1 108.0 mm to (162.3, 104.4)
- moved R10 107.9 mm to (157.0, 97.2)
- moved R11 107.9 mm to (154.0, 97.2)
- moved R8 107.9 mm to (163.0, 97.2)
- moved R9 107.9 mm to (160.0, 97.2)
- moved J5 101.0 mm to (165.0, 50.0), turned to -90 degrees
- moved Q1 100.7 mm to (191.0, 64.1)
- moved C4 100.2 mm to (192.0, 56.0), turned to 180 degrees
- moved C2 100.0 mm to (181.0, 50.0)
- moved R12 99.0 mm to (160.0, 118.0), turned to 0 degrees
- moved J2 97.6 mm to (181.0, 135.0), turned to 180 degrees
- moved J1 88.5 mm to (187.0, 135.0), turned to 180 degrees
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Routing:
- net /-R: track 0.00 -> 102.5 mm
- net VCC: track 0.00 -> 80.0 mm
- net Net-(Q2-B): track 0.00 -> 49.8 mm
- net /SW_OUT: track 0.00 -> 26.1 mm
- net Net-(JP1-A): track 0.00 -> 24.3 mm
- net Net-(D2-K): track 0.00 -> 20.6 mm
- net Net-(R9-Pad2): track 0.00 -> 18.1 mm
- net Net-(J4-P1): track 0.00 -> 8.27 mm
- net /V+: track 0.00 -> 7.10 mm
- net /+R: track 0.00 -> 7.06 mm
- net Net-(U1A--): track 0.00 -> 6.48 mm
- net Net-(U1A-+): track 0.00 -> 6.47 mm
- net Net-(D1-K): track 0.00 -> 4.00 mm

Commit message: new
Parts:
- added C6: 100n, Modified_Footprints:C_POL, F.Cu at (172.3, 114.3)
- added D3: RECTIFIER_DIODE, EESTN5:DO-41, F.Cu at (181.4, 121.6)
- added D4: RECTIFIER_DIODE, EESTN5:DO-41, F.Cu at (191.6, 59.6)
- moved Q5 23.6 mm to (194.2, 101.5)
- moved R7 21.9 mm to (195.4, 117.7), turned to -90 degrees
- moved R6 20.7 mm to (187.4, 135.5)
- moved SW1 16.4 mm to (156.6, 56.0)
- moved R5 16.0 mm to (163.8, 95.8), turned to 0 degrees
- moved R4 15.3 mm to (161.9, 77.6)
- moved R10 11.0 mm to (167.8, 99.4), turned to 180 degrees
- moved C1 10.6 mm to (181.5, 116.7)
- moved C3 10.3 mm to (189.6, 109.8)
- moved Q3 9.77 mm to (184.0, 101.3)
- moved R2 9.72 mm to (187.3, 128.9)
- moved R13 9.63 mm to (178.6, 102.2)
- moved R8 9.51 mm to (167.8, 105.4), turned to 180 degrees
- moved R9 9.37 mm to (167.8, 102.4), turned to 0 degrees
- moved JP3 9.36 mm to (171.4, 123.1), turned to 180 degrees
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Connections:
- R2 pad 1: /-R -> Net-(R2-Pad1)
- R2 pad 3: Net-(R2-Pad3) -> /-R
- R3 pad 1: Net-(R2-Pad3) -> Net-(JP1-A)
- R3 pad 3: Net-(JP1-A) -> Net-(R2-Pad1)
- U1 pad 8: VCC -> /SW_OUT
Routing:
- net /SW_OUT: track 26.1 -> 110.2 mm
- net /-R: track 102.5 -> 25.2 mm
- net Net-(JP1-A): track 24.3 -> 53.4 mm
- net Net-(Q2-B): track 49.8 -> 34.5 mm
- net Net-(JP2-B): track 0.00 -> 14.5 mm
- net Net-(JP1-B): track 0.00 -> 14.4 mm
- net /+R: track 7.06 -> 21.1 mm
- net Net-(J4-P1): track 8.27 -> 21.5 mm
- net Net-(U1A-+): track 6.47 -> 17.9 mm
- net VCC: track 80.0 -> 90.5 mm
- net Net-(Q3-B): track 0.00 -> 6.76 mm
- net Net-(R9-Pad2): track 18.1 -> 11.4 mm
- net Net-(Q4-E): track 0.00 -> 4.40 mm
- net Net-(D2-K): track 20.6 -> 23.7 mm
- net /V+: track 7.10 -> 4.56 mm
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
Commit message: new
Parts:
- moved C3 34.1 mm to (221.9, 120.6), turned to 0 degrees
- moved Q5 9.89 mm to (193.5, 111.4)
- moved JP1 4.03 mm to (183.2, 94.0)
- moved JP2 4.03 mm to (183.2, 97.5)
- moved R13 4.03 mm to (180.5, 105.8)
- moved R3 4.03 mm to (191.2, 94.0)
- moved Q3 4.03 mm to (185.9, 104.9)
- moved D3 3.82 mm to (178.6, 119.0), turned to -90 degrees
- moved R7 3.37 mm to (192.3, 119.0), turned to 0 degrees
- moved C1 3.12 mm to (183.5, 119.1), turned to 90 degrees
- moved C6 1.60 mm to (170.7, 114.2)
- moved SW2 0.90 mm to (163.3, 133.1)
- moved JP3 0.82 mm to (171.6, 123.9)
- moved J4 0.12 mm to (162.5, 127.6)
- moved R2 0.10 mm to (187.3, 129.0)
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Connections:
- SW2 pad 1: Net-(R9-Pad2) -> /V+
- SW2 pad 2: /V+ -> Net-(R9-Pad2)
Routing:
- net /-R: track 25.2 -> 94.7 mm
- net Net-(JP1-A): track 53.4 -> 111.4 mm
- net Net-(Q2-B): track 34.5 -> 76.2 mm
- net Net-(R2-Pad1): track 0.00 -> 37.5 mm
- net Net-(JP2-B): track 14.5 -> 38.2 mm
- net Net-(R6-Pad2): track 0.00 -> 21.5 mm
- net Net-(Q3-B): track 6.76 -> 18.7 mm
- net /+R: track 21.1 -> 15.6 mm
- net /SW_OUT: track 110.2 -> 108.6 mm
- net Net-(J4-P1): track 21.5 -> 20.8 mm
