File: Power_Supply/Power_Supply.kicad_sch (KiCad schematic)
At the start: 28 parts, among them J1 TB_1X2, J2 TB_1X2, J3 CONN_01X03, J4 CONN_01X03, Q1 TIP41C, Q2 BD139, Q3 BC548, Q4 BC558, Q5 BC558, U1 LM358

Commit message: new
Parts:
- removed J1, J2: TB_1X2, symbol EESTN5:TB_1X2
- added J1, J2: Cable_PAD, EESTN5:Cable_1,5mm, symbol EESTN5:Cable_PAD
- added J5: jack, MacroLib:Jack_hembra_DC_barrel, symbol MacroLib:jack
- D1, D2: footprint (none) -> EESTN5:DO-41
- J3, J4: footprint (none) -> EESTN5:Pin_Header_3
- Q1: footprint (none) -> EESTN5:TO-220
- Q2: footprint BD139 -> (none)
- Q3: footprint EESTN5:TO-92 -> EESTN5:to92
- Q4, Q5: footprint 3-LEAD_TO-92_AMMO -> EESTN5:to92
- R1, R10, R11, R12, R4, R5, R7, R8, R9: footprint (none) -> EESTN5:RES0.3
- R2, R6: footprint (none) -> EESTN5:Potenciometro
- U1: footprint (none) -> EESTN5:DIP-8
Connections:
- net -R: now also J1.1
- net GND: now also J4.3 (P3), J2.1, J5.2, J5.3
- net VCC: now also J4.2 (P2), J5.1
- net V+: now reaches J3.2 (P2)
- net V+: now also J4.1 (P1)
Other:
- moved on the sheet: J4

Commit message: new footprint
Parts:
- Q1: footprint EESTN5:TO-220 -> Modified_Footprints:TO-220-3_Vertical
Changed lines of the file:
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@@
 			)
 		)
-		(property "Footprint" "EESTN5:TO-220"
+		(property "Footprint" "Modified_Footprints:TO-220-3_Vertical"
 			(at 176.53 168.58 0)
 			(effects

Commit message: new
Parts:
- removed J3: CONN_01X03, EESTN5:Pin_Header_3, symbol EESTN5:CONN_01X03
- added JP1, JP2: Jumper, symbol EESTN5:Jumper
- added SW1: SW_SPST, symbol SW:SW_SPST
- added SW2: SW_Push, symbol SW:SW_Push
- added unit 2 of U1
Connections:
- net +R: now also R10.1; no longer R8.1
- net -R: now also R12.2, R8.1; no longer R10.1
- net GND: now also SW2.3
- net V+: now also R12.1, SW2.2, U1.5 (+); no longer J4.1 (P1)
- net VCC: now also SW1.1 (A); no longer J5.1
- net at R9.2, U1.1: now also SW2.1; no longer R12.1
- net at Q1.1 (B), Q2.1 (E), Q5.3 (E)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: now also JP1.1 (A); no longer R3.2
- net at Q5.2 (B), R2.2: now also JP2.2 (B)
- new net: JP1.2 (B), JP2.1 (A), R3.2
- new net: J4.1 (P1), U1.6 (-), U1.7
- new net: J5.1, SW1.2 (B)
Other:
- moved on the sheet: C1, C2, C3, C4, J1, J2, J4, Q1, Q3, Q5, R1, R10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

Commit message: new
Parts:
- added C5: 10uf, EESTN5:CAP_ELEC_5x11mm, symbol EESTN5:C
- added R13: 1M, EESTN5:RES0.3, symbol EESTN5:R
- C1, C4: value C -> 100nf; footprint (none) -> Modified_Footprints:C_POL
- C2: value C -> 2200uf; footprint (none) -> Modified_Footprints:C_ELEC_15x12
- C3: value C -> 470uf; footprint (none) -> Modified_Footprints:C-ELEC
- JP1, JP2: footprint (none) -> Modified_Footprints:JUMPER
- Q1: footprint Modified_Footprints:TO-220-3_Vertical -> Modified_Footprints:TO-220-3_90
- Q2: footprint (none) -> Modified_Footprints:TO-126-3_90
- R1: value R -> 0R2; footprint EESTN5:RES0.3 -> Modified_Footprints:RESO_2W
- R10, R8: value R -> 1k1
- R11, R9: value R -> 5k6
- R12: value R -> 100k
- R3: footprint (none) -> EESTN5:TRIMER_V
- R4: value R -> 100
- R5: value R -> 10k
- R7: value R -> 2k2
- SW1: footprint (none) -> EESTN5:BORNERA2
- SW2: footprint (none) -> MacroLib:PUSH_SWITCH_THT_90
- U1: footprint (none) -> EESTN5:DIP-8
Connections:
- net GND: now also C5.2, R13.2
- net VCC: now also J5.1, SW1.2 (B); no longer D1.1 (A), J4.2 (P2), R4.1, SW1.1 (A)
- net at D2.2 (K), Q4.2 (B), R5.1: now also C5.1
- net at Q2.3 (B), Q3.1 (C), Q4.1 (C): now also R13.1
- new net SW_OUT: D1.1 (A), J4.2 (P2), R4.1, SW1.1 (A)
Other:
- moved on the sheet: C2, C4, D1, D2, J4, R5, SW1, U1B

Commit message: new
Parts:
- added J3, J6, J7, J8: Cable_PAD, EESTN5:Separador_M3_10mm, symbol EESTN5:Cable_PAD
- added JP3: Jumper, Modified_Footprints:JUMPER, symbol EESTN5:Jumper
- R2, R6: footprint EESTN5:Potenciometro -> EESTN5:Pin_Header_3
- SW1: footprint EESTN5:BORNERA2 -> EESTN5:Pin_Header_2
Connections:
- net -R: now also JP3.1 (A)
- net at J4.1 (P1), U1.6 (-), U1.7: now also JP3.2 (B)

Commit message: new
Parts:
- added C6: 100n, Modified_Footprints:C_POL, symbol EESTN5:C
- added D3, D4: RECTIFIER_DIODE, EESTN5:DO-41, symbol Diodes:RECTIFIER_DIODE
Connections:
- net +R: now also D4.1 (A)
- net -R: now also R2.3, D3.2 (K); no longer R2.1
- net GND: now also C6.2, D3.1 (A)
- net SW_OUT: now also U1.8 (+), C6.1
- net VCC: now also D4.2 (K); no longer U1.8 (+)
- net at JP1.1 (A), Q1.1 (B), Q2.1 (E)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: now also R3.1; no longer R3.3
- new net: R2.1, R3.3

Commit message: new
Connections:
- net V+: now also SW2.1; no longer SW2.2
- net at R9.2, U1.1: now also SW2.2; no longer SW2.1
Changed lines of the file:
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@@
 		(lib_id "SW:SW_Push")
 		(at 246.38 139.7 0)
+		(mirror y)
 		(unit 1)
 		(exclude_from_sim no)
@@
 		(on_board yes)
 		(dnp no)
-		(fields_autoplaced yes)
 		(property "Reference" "SW2"
 			(at 246.38 134.62 0)
@@
 		)
 		(property "Value" "SW_Push"
-			(at 254 142.494 0)
+			(at 238.76 142.494 0)
 			(effects
 				(font
@@
 		)
 		(property "Description" "Push button switch, generic, two pins"
-			(at 268.224 144.272 0)
+			(at 224.536 144.272 0)
 			(effects
 				(font
